File: input-board.kicad_pcb (KiCad board)
At the start: 2 copper layers, 87.5 x 28.2 mm, 72 parts, among them J1 BTNCON, J12 CAN, J2 BTNCON, J3 SWD, J7 I2C, J8 GAS, J9 BREMSE, SW1 switch-with-led, SW2 switch-with-led, SW3 switch-with-led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

Commit message: Layout prelim done
Routing:
- net +3V3: track 71.6 -> 137.4 mm, vias 4 -> 6
- net SWCLK: track 0.00 -> 17.5 mm, vias 0 -> 2
- net RAW_GAS: track 4.76 -> 21.4 mm, vias 0 -> 2
- net RAW_BREMSE: track 4.76 -> 19.3 mm, vias 0 -> 2
- net SWDIO: track 0.00 -> 14.1 mm
- net Net-(U2-Pad5): track 0.00 -> 9.44 mm, vias 0 -> 2
- net MDLED2: track 17.8 -> 19.7 mm, vias 1 -> 2
- net Net-(U1-Pad4): track 0.00 -> 1.60 mm
- net MDBT4: track 33.2 -> 31.9 mm
- net MDLED4: track 51.2 -> 50.1 mm
- net MDBT1: track 32.2 -> 31.2 mm
- net BTN5: track 32.8 -> 31.8 mm
- net MDLED1: track 46.8 -> 46.1 mm
- net MDLED3: vias 1 -> 2
- net Net-(J9-Pad2): vias 0 -> 1
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Other:
- board size 87.5 x 28.2 mm -> 86.5 x 27.8 mm
- board text added: "15V CANH CANL GND"
- board text added: "3V3 BREMS GND"
- board text added: "GND B3 B2 B1"
- board text added: "GND B6 B5 B4"
- board text added: "GND CLK IO 3V3"
- board text added: "GND GAS 3V3"
- board text added: "GND SDA 3V3 SCL"

Commit message: Added input reverse protection
Parts:
- added D9: D_Schottky, Diode_SMD:D_SOD-123, F.Cu at (140.0, 41.2)
- moved R25 1.01 mm to (140.4, 38.0), turned to 180 degrees
Connections:
- J12 pad 1: 15V -> Net-(D9-Pad2)
- U1 pad 10: (no net) -> Net-(U1-Pad10)
- U1 pad 11: (no net) -> Net-(U1-Pad11)
- U1 pad 15: (no net) -> Net-(U1-Pad15)
- U1 pad 18: (no net) -> Net-(U1-Pad18)
- U1 pad 2: (no net) -> Net-(U1-Pad2)
- U2 pad 1: (no net) -> Net-(U2-Pad1)
- U2 pad 12: (no net) -> Net-(U2-Pad12)
- U2 pad 13: (no net) -> Net-(U2-Pad13)
- U2 pad 14: (no net) -> Net-(U2-Pad14)
- U2 pad 15: (no net) -> Net-(U2-Pad15)
- U2 pad 16: (no net) -> Net-(U2-Pad16)
- U2 pad 17: (no net) -> Net-(U2-Pad17)
- U2 pad 2: (no net) -> Net-(U2-Pad2)
- U2 pad 3: (no net) -> Net-(U2-Pad3)
- U2 pad 30: (no net) -> Net-(U2-Pad30)
- U2 pad 31: (no net) -> Net-(U2-Pad31)
- U2 pad 4: (no net) -> Net-(U2-Pad4)
- U2 pad 41: (no net) -> Net-(U2-Pad41)
- U2 pad 6: (no net) -> Net-(U2-Pad6)
Routing:
- net Net-(D9-Pad2): track 0.00 -> 5.08 mm
- net 15V: track 12.1 -> 14.7 mm
- net Net-(R25-Pad2): track 2.14 -> 2.82 mm
- net Net-(U2-Pad5): track 9.44 -> 8.78 mm

Commit message: Changed input to LDO Added JLCPCB #
Parts:
- removed R1: 100k, Resistor_SMD:R_0603_1608Metric
- removed R12: 30.1k, Resistor_SMD:R_0603_1608Metric
- removed R3: 160k, Resistor_SMD:R_0603_1608Metric
- C4: value 22uF -> 10uF
- U1: value MPM3620 -> L7805; footprint boardcomputer:QFN-20-1EP_3x5mm_P0.85mm -> Package_TO_SOT_SMD:SOT-223-3_TabPin2
- moved C4 3.95 mm to (157.0, 39.8), turned to 270 degrees
- moved C3 0.50 mm to (149.2, 43.5)
- moved U1 0.50 mm to (153.8, 43.5)
Connections:
- U1 pad 1: Net-(R12-Pad2) -> 15V
- U1 pad 2: Net-(U1-Pad2) -> GND
- U1 pad 3: GND -> +5V
- U2 pad 1: Net-(U2-Pad1) -> (no net)
- U2 pad 12: Net-(U2-Pad12) -> (no net)
- U2 pad 13: Net-(U2-Pad13) -> (no net)
- U2 pad 14: Net-(U2-Pad14) -> (no net)
- U2 pad 15: Net-(U2-Pad15) -> (no net)
- U2 pad 16: Net-(U2-Pad16) -> (no net)
- U2 pad 17: Net-(U2-Pad17) -> (no net)
- U2 pad 2: Net-(U2-Pad2) -> (no net)
- U2 pad 3: Net-(U2-Pad3) -> (no net)
- U2 pad 30: Net-(U2-Pad30) -> (no net)
- U2 pad 31: Net-(U2-Pad31) -> (no net)
- U2 pad 4: Net-(U2-Pad4) -> (no net)
- U2 pad 41: Net-(U2-Pad41) -> (no net)
- U2 pad 6: Net-(U2-Pad6) -> (no net)
Routing:
- net Net-(R12-Pad2): track 7.61 -> 0.00 mm
- net GND: track 17.3 -> 10.6 mm, vias 260 -> 271
- net Net-(R1-Pad1): track 2.56 -> 0.00 mm
- net +5V: track 62.0 -> 64.1 mm
- net 15V: track 14.7 -> 13.0 mm
- net Net-(U1-Pad4): track 1.60 -> 0.00 mm

Commit message: Added nc to unused pins
Parts:
- D9: value D_Schottky -> B5819W
- R11, R17, R18, R19, R20, R21, R22, R23, R24: value 10k -> 10K
- R15, R16: value 4k7 -> 4K7
- R2, R4: value PULLDOWN -> 10K
- R25: value 100k -> 100K
- R48, R49: value 60R -> 56R
- U1: value L7805 -> UA78M05IDCYR
Connections:
- net 15V renamed +15V
